Commit message: base_footprint is now the root in URDF

File: src/description/zuuu_description.urdf.xacro (robot description, xacro)
@@ -1,4 +1,6 @@
 <?xml version="1.0"?>
 <robot name="zuuu" xmlns:xacro="http://ros.org/wiki/xacro">
+  <!-- omni_steering -->
+	<!-- <xacro:include filename="/home/remi/ros2_ws/src/zuuu_description/src/description/zuuu_omni_steering.urdf.xacro" /> -->
   <!-- Define robot constants -->
   <xacro:property name="base_radius" value="0.16"/>
@@ -30,4 +32,13 @@
     </inertial>
   </xacro:macro>
+  <!-- Robot Footprint -->
+  <link name="base_footprint"/>
+  <joint name="base_footprint_joint" type="fixed">
+    <origin rpy="0 0 0" xyz="0 0 0"/>
+    <axis xyz="0 0 ${(base_top_height-base_depth/2)}"/>
+    <joint_properties damping="1" friction="1"/>
+    <parent link="base_footprint"/>
+    <child link="base_link"/>
+  </joint>
   <!-- Robot Base -->
   <link name="base_link">
@@ -47,13 +58,4 @@
     <xacro:cylinder_inertia m="20" r="${base_radius}" h="${base_depth}"/>
   </link>
-   <!-- Robot Footprint -->
-  <link name="base_footprint">
-  	<xacro:box_inertia m="0" w="0" d="0" h="0"/>
-  </link>
-  <joint name="base_joint" type="fixed">
-    <parent link="base_link"/>
-    <child link="base_footprint"/>
-    <origin xyz="0.0 0.0 ${-(base_top_height-base_depth/2)}" rpy="0 0 0"/>
-  </joint>
   <!-- Wheels -->
   <xacro:macro name="wheel" params="prefix yaw_angle">
@@ -76,4 +78,5 @@
       <xacro:cylinder_inertia m="0.5" r="${wheel_radius}" h="${wheel_width}"/>
     </link>
+<!-- I've seen a robot using "fixed" instead of continuous here. Tried it but the robot has a weird behaviour and falls down (kinda expected). But with continuous the TF doesn't appear. -->
     <joint name="${prefix}_joint" type="continuous">
       <parent link="base_link"/>
@@ -87,4 +90,67 @@
   <xacro:wheel prefix="drivewhl2" yaw_angle="${5*pi/3}" />
   <xacro:wheel prefix="drivewhl3" yaw_angle="${pi}" />
+  <!-- Doesn't seem to be working well (tf not being published?), so I'm doing it by hand -->
+  <transmission name="drivewhl1">
+    <type>transmission_interface/SimpleTransmission</type>
+    <joint name="drivewhl1_joint">
+      <hardwareInterface>hardware_interface/VelocityJointInterface</hardwareInterface>
+    </joint>
+    <actuator name="drivewhl1_motor">
+      <mechanicalReduction>1</mechanicalReduction>
+    </actuator>
+  </transmission>
+  <transmission name="drivewhl2">
+    <type>transmission_interface/SimpleTransmission</type>
+    <joint name="drivewhl2_joint">
+      <hardwareInterface>hardware_interface/VelocityJointInterface</hardwareInterface>
+    </joint>
+    <actuator name="drivewhl2_motor">
+      <mechanicalReduction>1</mechanicalReduction>
+    </actuator>
+  </transmission>
+  <transmission name="drivewhl3">
+    <type>transmission_interface/SimpleTransmission</type>
+    <joint name="drivewhl3_joint">
+      <hardwareInterface>hardware_interface/VelocityJointInterface</hardwareInterface>
+    </joint>
+    <actuator name="drivewhl3_motor">
+      <mechanicalReduction>1</mechanicalReduction>
+    </actuator>
+  </transmission>
+  <!-- <xacro:macro name="omni_steering" params="">
+    <gazebo>
+      <plugin name="omni_steering" filename="libgazebo_ros_planar_move.so">
+        <commandTopic>cmd_vel</commandTopic>
+        <odometryTopic>odom</odometryTopic>
+        <odometryFrame>odom</odometryFrame>
+        <odometryRate>50.0</odometryRate>
+        <robotBaseFrame>base_link</robotBaseFrame>
+        <publishTF>true</publishTF>
+      </plugin>
+    </gazebo>
+  </xacro:macro> -->
+  <!-- <xacro:omni_steering/> -->
+  <gazebo>
+    <plugin name="object_controller" filename="libgazebo_ros_planar_move.so">
+      <commandTopic>cmd_vel</commandTopic>
+      <odometryTopic>odom</odometryTopic>
+      <robotNamespace><remapping>/tf:=tf</remapping>  </robotNamespace>
+      <ros>    <remapping>/tf:=tf</remapping>    </ros>
+      <!-- Set control loop update rate -->
+      <odometryRate>100</odometryRate>
+      <!-- Set odom publish rate -->
+      <publish_rate>100</publish_rate>
+      <!-- Set if odom required -->
+      <publish_odom>true</publish_odom>
+      <publish_odom_tf>true</publish_odom_tf>
+      <!-- Frame IDs -->
+      <odometryFrame>odom</odometryFrame>
+      <robotBaseFrame>base_link</robotBaseFrame>
+      <!-- Set odom covariance -->
+      <covariance_x>0.0001</covariance_x>
+      <covariance_y>0.0001</covariance_y>
+      <covariance_yaw>0.01</covariance_yaw>
+    </plugin>
+  </gazebo>
   <link name="imu_link">
     <visual>
@@ -298,3 +364,8 @@
     </sensor>
   </gazebo>
+  <gazebo>
+      <plugin name="gazebo_ros2_control" filename="libgazebo_ros2_control.so">
+        <parameters>$(find zuuu_description)/config/zuuu_controllers.yaml</parameters>
+      </plugin>
+  </gazebo>
 </robot>

Commit message: Adding friction parameters to handle holo wheels with physics

File: src/description/zuuu_description.urdf.xacro (robot description, xacro)
@@ -11,4 +11,6 @@
   <xacro:property name="wheel_radial_dist" value="0.1805"/>
   <xacro:property name="wheel_zoff" value="0.20"/>
+  <xacro:property name="global_damping" value="1.0"/>
+  <xacro:property name="global_friction" value="1.0"/>
   <!-- Define some commonly used intertial properties  -->
   <xacro:macro name="box_inertia" params="m w h d">
@@ -37,5 +39,5 @@
     <origin rpy="0 0 0" xyz="0 0 0"/>
     <axis xyz="0 0 ${(base_top_height-base_depth/2)}"/>
-    <joint_properties damping="1" friction="1"/>
+    <!-- <joint_properties damping="${global_damping}" friction="${global_friction}"/> -->
     <parent link="base_footprint"/>
     <child link="base_link"/>
@@ -64,9 +66,8 @@
         <origin xyz="0 0 0" rpy="${pi/2} 0 0"/>
         <geometry>
-            <cylinder radius="${wheel_radius}" length="${wheel_width}"/>
+            <box size="${wheel_radius} ${wheel_radius} ${wheel_width}"/>
+            <!-- <cylinder radius="${wheel_radius}" length="${wheel_width}"/> -->
         </geometry>
-        <material name="Gray">
-          <color rgba="0.5 0.5 0.5 1.0"/>
-        </material>
+        <material name="Bricks"></material>
       </visual>
       <collision>
@@ -84,5 +85,15 @@
       <origin xyz="${wheel_radial_dist*cos(yaw_angle)} ${-wheel_radial_dist*sin(yaw_angle)} ${-((base_top_height-base_depth/2)- wheel_radius)}" rpy="0 0 ${pi/2-yaw_angle}"/>
       <axis xyz="0 1 0"/>
+      <joint_properties damping="${global_damping}" friction="${global_friction}"/>
+      <limit effort="100" velocity="100"/>
     </joint>
+    <gazebo reference="${prefix}_link">
+      <mu1 value="1.0"/>
+      <mu2 value="0.0"/>
+      <kp value="10000000.0" />
+      <kd value="1.0" />
+      <fdir1 value="1 0 0"/>
+          <turnGravityOff>false</turnGravityOff>
+    </gazebo>
   </xacro:macro>
   <!-- Wheel 1 at the back, 2 on the right, 3 on the left -->
@@ -118,23 +129,9 @@
     </actuator>
   </transmission>
-  <!-- <xacro:macro name="omni_steering" params="">
-    <gazebo>
-      <plugin name="omni_steering" filename="libgazebo_ros_planar_move.so">
-        <commandTopic>cmd_vel</commandTopic>
-        <odometryTopic>odom</odometryTopic>
-        <odometryFrame>odom</odometryFrame>
-        <odometryRate>50.0</odometryRate>
-        <robotBaseFrame>base_link</robotBaseFrame>
-        <publishTF>true</publishTF>
-      </plugin>
-    </gazebo>
-  </xacro:macro> -->
-  <!-- <xacro:omni_steering/> -->
   <gazebo>
     <plugin name="object_controller" filename="libgazebo_ros_planar_move.so">
       <commandTopic>cmd_vel</commandTopic>
       <odometryTopic>odom</odometryTopic>
-      <robotNamespace><remapping>/tf:=tf</remapping>  </robotNamespace>
-      <ros>    <remapping>/tf:=tf</remapping>    </ros>
+      <robotNamespace> </robotNamespace>
       <!-- Set control loop update rate -->
       <odometryRate>100</odometryRate>

Commit message: Working version with ros2_control handling the joint state broadcast. This was hell and I hate everything and everybody

File: src/description/zuuu_description.urdf.xacro (robot description, xacro)
@@ -101,32 +101,4 @@
   <xacro:wheel prefix="drivewhl2" yaw_angle="${5*pi/3}" />
   <xacro:wheel prefix="drivewhl3" yaw_angle="${pi}" />
-  <!-- Doesn't seem to be working well (tf not being published?), so I'm doing it by hand -->
-  <transmission name="drivewhl1">
-    <type>transmission_interface/SimpleTransmission</type>
-    <joint name="drivewhl1_joint">
-      <hardwareInterface>hardware_interface/VelocityJointInterface</hardwareInterface>
-    </joint>
-    <actuator name="drivewhl1_motor">
-      <mechanicalReduction>1</mechanicalReduction>
-    </actuator>
-  </transmission>
-  <transmission name="drivewhl2">
-    <type>transmission_interface/SimpleTransmission</type>
-    <joint name="drivewhl2_joint">
-      <hardwareInterface>hardware_interface/VelocityJointInterface</hardwareInterface>
-    </joint>
-    <actuator name="drivewhl2_motor">
-      <mechanicalReduction>1</mechanicalReduction>
-    </actuator>
-  </transmission>
-  <transmission name="drivewhl3">
-    <type>transmission_interface/SimpleTransmission</type>
-    <joint name="drivewhl3_joint">
-      <hardwareInterface>hardware_interface/VelocityJointInterface</hardwareInterface>
-    </joint>
-    <actuator name="drivewhl3_motor">
-      <mechanicalReduction>1</mechanicalReduction>
-    </actuator>
-  </transmission>
   <gazebo>
     <plugin name="object_controller" filename="libgazebo_ros_planar_move.so">
@@ -148,4 +120,40 @@
       <covariance_y>0.0001</covariance_y>
       <covariance_yaw>0.01</covariance_yaw>
+    </plugin>
+  </gazebo>
+  <ros2_control name="GazeboSystem" type="system">
+    <hardware>
+        <plugin>gazebo_ros2_control/GazeboSystem</plugin>
+        <!-- <plugin>fake_components/GenericSystem</plugin> -->
+    </hardware>
+    <joint name="drivewhl1_joint">
+      <command_interface name="velocity">
+          <param name="min">-1</param>
+          <param name="max">1</param>
+        </command_interface>
+        <state_interface name="position"/>
+        <state_interface name="velocity"/>
+    </joint>
+    <joint name="drivewhl2_joint">
+      <command_interface name="velocity">
+          <param name="min">-1</param>
+          <param name="max">1</param>
+        </command_interface>
+        <state_interface name="position"/>
+        <state_interface name="velocity"/>
+    </joint>
+    <joint name="drivewhl3_joint">
+      <command_interface name="velocity">
+          <param name="min">-1</param>
+          <param name="max">1</param>
+        </command_interface>
+        <state_interface name="position"/>
+        <state_interface name="velocity"/>
+    </joint>
+  </ros2_control>
+  <!-- Calling the pluging that will parse the ros2_control tags -->
+  <gazebo>
+    <plugin filename="libgazebo_ros2_control.so" name="gazebo_ros2_control">
+      <parameters>$(find zuuu_description)/config/zuuu_controllers.yaml</parameters>
     </plugin>
   </gazebo>
@@ -361,8 +369,3 @@
     </sensor>
   </gazebo>
-  <gazebo>
-      <plugin name="gazebo_ros2_control" filename="libgazebo_ros2_control.so">
-        <parameters>$(find zuuu_description)/config/zuuu_controllers.yaml</parameters>
-      </plugin>
-  </gazebo>
 </robot>

Commit message: We can see round wheels turning now

File: src/description/zuuu_description.urdf.xacro (robot description, xacro)
@@ -11,6 +11,6 @@
   <xacro:property name="wheel_radial_dist" value="0.1805"/>
   <xacro:property name="wheel_zoff" value="0.20"/>
-  <xacro:property name="global_damping" value="1.0"/>
-  <xacro:property name="global_friction" value="1.0"/>
+  <xacro:property name="global_damping" value="0.5"/>
+  <xacro:property name="global_friction" value="0.5"/>
   <!-- Define some commonly used intertial properties  -->
   <xacro:macro name="box_inertia" params="m w h d">
@@ -66,6 +66,6 @@
         <origin xyz="0 0 0" rpy="${pi/2} 0 0"/>
         <geometry>
-            <box size="${wheel_radius} ${wheel_radius} ${wheel_width}"/>
-            <!-- <cylinder radius="${wheel_radius}" length="${wheel_width}"/> -->
+            <cylinder radius="${wheel_radius}" length="${wheel_width}"/>
+            <box size="${wheel_radius} ${wheel_radius} ${wheel_width+0.02}"/>
         </geometry>
         <material name="Bricks"></material>
@@ -79,5 +79,5 @@
       <xacro:cylinder_inertia m="0.5" r="${wheel_radius}" h="${wheel_width}"/>
     </link>
-<!-- I've seen a robot using "fixed" instead of continuous here. Tried it but the robot has a weird behaviour and falls down (kinda expected). But with continuous the TF doesn't appear. -->
+    <!-- I've seen a robot using "fixed" instead of continuous here...-->
     <joint name="${prefix}_joint" type="continuous">
       <parent link="base_link"/>
@@ -86,6 +86,6 @@
       <axis xyz="0 1 0"/>
       <joint_properties damping="${global_damping}" friction="${global_friction}"/>
-      <limit effort="100" velocity="100"/>
-    </joint>
+    </joint>
+    <!-- Physics! -->
     <gazebo reference="${prefix}_link">
       <mu1 value="1.0"/>
@@ -94,6 +94,23 @@
       <kd value="1.0" />
       <fdir1 value="1 0 0"/>
-          <turnGravityOff>false</turnGravityOff>
+      <maxVel>1.0</maxVel>
+      <minDepth>0.0</minDepth>
+      <turnGravityOff>false</turnGravityOff>
     </gazebo>
+    <!-- Just so that we can see the wheels turn -->
+    <link name="${prefix}_extra_link">
+      <visual>
+        <origin xyz="0 0 0" rpy="${pi/2} 0 0"/>
+        <geometry>
+            <box size="${wheel_radius} ${wheel_radius} ${wheel_width+0.02}"/>
+        </geometry>
+      </visual>
+    </link>
+    <joint name="${prefix}_extra_joint" type="fixed">
+      <origin rpy="0 0 0" xyz="0 0 0"/>
+      <axis xyz="0 0 0"/>
+      <parent link="${prefix}_link"/>
+      <child link="${prefix}_extra_link"/>
+    </joint>
   </xacro:macro>
   <!-- Wheel 1 at the back, 2 on the right, 3 on the left -->

Commit message: boolean flag for the fixed wheels hack

File: src/description/zuuu_description.urdf.xacro (robot description, xacro)
@@ -1,5 +1,6 @@
 <?xml version="1.0"?>
 <robot name="zuuu" xmlns:xacro="http://ros.org/wiki/xacro">
-  <xacro:arg name="use_fake_components" default="true"/>
+  <xacro:arg name="use_fake_components" default="false"/>
+  <xacro:arg name="use_fixed_wheels" default="true"/>
   <!-- Define robot constants -->
   <xacro:property name="base_radius" value="0.16"/>
@@ -78,24 +79,45 @@
       <xacro:cylinder_inertia m="0.5" r="${wheel_radius}" h="${wheel_width}"/>
     </link>
-    <!-- I've seen a robot using "fixed" instead of continuous here...-->
-    <joint name="${prefix}_joint" type="continuous">
-      <parent link="base_link"/>
-      <child link="${prefix}_link"/>
-      <origin xyz="${wheel_radial_dist*cos(yaw_angle)} ${-wheel_radial_dist*sin(yaw_angle)} ${-((base_top_height-base_depth/2)- wheel_radius)}" rpy="0 0 ${pi/2-yaw_angle}"/>
-      <axis xyz="0 1 0"/>
-      <joint_properties damping="${global_damping}" friction="${global_friction}"/>
-    </joint>
-    <!-- Physics! -->
-    <gazebo reference="${prefix}_link">
-      <mu1 value="1.0"/>
-      <mu2 value="0.0"/>
-      <kp value="10000000.0" />
-      <kd value="1.0" />
-      <fdir1 value="1 0 0"/>
-      <maxVel>1.0</maxVel>
-      <minDepth>0.0</minDepth>
-      <turnGravityOff>false</turnGravityOff>
-    </gazebo>
-    <!-- Just so that we can see the wheels turn -->
+    <xacro:if value="$(arg use_fixed_wheels)">
+        <joint name="${prefix}_joint" type="fixed">
+          <parent link="base_link"/>
+          <child link="${prefix}_link"/>
+          <origin xyz="${wheel_radial_dist*cos(yaw_angle)} ${-wheel_radial_dist*sin(yaw_angle)} ${-((base_top_height-base_depth/2)- wheel_radius)}" rpy="0 0 ${pi/2-yaw_angle}"/>
+          <axis xyz="0 1 0"/>
+          <joint_properties damping="${global_damping}" friction="${global_friction}"/>
+        </joint>
+        <!-- No friction because we suck and everything is lame -->
+        <gazebo reference="${prefix}_link">
+          <mu1 value="0.0"/>
+          <mu2 value="0.0"/>
+          <kp value="10000000.0" />
+          <kd value="1.0" />
+          <fdir1 value="1 0 0"/>
+          <maxVel>1.0</maxVel>
+          <minDepth>0.0</minDepth>
+          <turnGravityOff>false</turnGravityOff>
+        </gazebo>
+    </xacro:if>
+    <xacro:unless value="$(arg use_fixed_wheels)">
+      <joint name="${prefix}_joint" type="continuous">
+        <parent link="base_link"/>
+        <child link="${prefix}_link"/>
+        <origin xyz="${wheel_radial_dist*cos(yaw_angle)} ${-wheel_radial_dist*sin(yaw_angle)} ${-((base_top_height-base_depth/2)- wheel_radius)}" rpy="0 0 ${pi/2-yaw_angle}"/>
+        <axis xyz="0 1 0"/>
+        <joint_properties damping="${global_damping}" friction="${global_friction}"/>
+      </joint>
+      <!-- Physics because we're smart and handsome -->
+      <gazebo reference="${prefix}_link">
+        <mu1 value="1.0"/>
+        <mu2 value="0.0"/>
+        <kp value="10000000.0" />
+        <kd value="1.0" />
+        <fdir1 value="1 0 0"/>
+        <maxVel>5.0</maxVel>
+        <minDepth>0.002</minDepth>
+        <turnGravityOff>false</turnGravityOff>
+      </gazebo>
+    </xacro:unless>
+    <!-- Just so that we can see the wheels turn when they turn -->
     <link name="${prefix}_extra_link">
       <visual>

Commit message: hopeless friction tuning

File: src/description/zuuu_description.urdf.xacro (robot description, xacro)
@@ -12,5 +12,5 @@
   <xacro:property name="wheel_zoff" value="0.20"/>
   <xacro:property name="global_damping" value="0.5"/>
-  <xacro:property name="global_friction" value="0.5"/>
+  <xacro:property name="global_friction" value="0.1"/>
   <!-- Define some commonly used intertial properties  -->
   <xacro:macro name="box_inertia" params="m w h d">

Commit message: minor fixes and use_sim_time debug wip

File: src/description/zuuu_description.urdf.xacro (robot description, xacro)
@@ -3,4 +3,5 @@
   <xacro:arg name="use_fake_components" default="false"/>
   <xacro:arg name="use_fixed_wheels" default="true"/>
+  <xacro:arg name="use_ros_control" default="false"/>
   <!-- Define robot constants -->
   <xacro:property name="base_radius" value="0.16"/>
@@ -160,46 +161,48 @@
     </plugin>
   </gazebo>
-  <ros2_control name="zuuu_ros2_control" type="system">
-    <hardware>
-      <xacro:if value="$(arg use_fake_components)">
-        <plugin>fake_components/GenericSystem</plugin>
-      </xacro:if>
-      <xacro:unless value="$(arg use_fake_components)">
-        <plugin>gazebo_ros2_control/GazeboSystem</plugin>
-      </xacro:unless>
-    </hardware>
-    <joint name="drivewhl1_joint">
-      <command_interface name="velocity">
-          <param name="min">-1</param>
-          <param name="max">1</param>
-        </command_interface>
-        <state_interface name="position"/>
-        <state_interface name="velocity"/>
-    </joint>
-    <joint name="drivewhl2_joint">
-      <command_interface name="velocity">
-          <param name="min">-1</param>
-          <param name="max">1</param>
-        </command_interface>
-        <state_interface name="position"/>
-        <state_interface name="velocity"/>
-    </joint>
-    <joint name="drivewhl3_joint">
-      <command_interface name="velocity">
-          <param name="min">-1</param>
-          <param name="max">1</param>
-        </command_interface>
-        <state_interface name="position"/>
-        <state_interface name="velocity"/>
-    </joint>
-  </ros2_control>
-  <!-- Calling the pluging that will parse the ros2_control tags -->
-  <xacro:unless value="$(arg use_fake_components)">
-    <gazebo>
-      <plugin filename="libgazebo_ros2_control.so" name="gazebo_ros2_control">
-        <parameters>$(find zuuu_description)/config/zuuu_controllers.yaml</parameters>
-      </plugin>
-    </gazebo>
-  </xacro:unless>
+  <xacro:if value="$(arg use_ros_control)">
+    <ros2_control name="zuuu_ros2_control" type="system">
+      <hardware>
+        <xacro:if value="$(arg use_fake_components)">
+          <plugin>fake_components/GenericSystem</plugin>
+        </xacro:if>
+        <xacro:unless value="$(arg use_fake_components)">
+          <plugin>gazebo_ros2_control/GazeboSystem</plugin>
+        </xacro:unless>
+      </hardware>
+      <joint name="drivewhl1_joint">
+        <command_interface name="velocity">
+            <param name="min">-1</param>
+            <param name="max">1</param>
+          </command_interface>
+          <state_interface name="position"/>
+          <state_interface name="velocity"/>
+      </joint>
+      <joint name="drivewhl2_joint">
+        <command_interface name="velocity">
+            <param name="min">-1</param>
+            <param name="max">1</param>
+          </command_interface>
+          <state_interface name="position"/>
+          <state_interface name="velocity"/>
+      </joint>
+      <joint name="drivewhl3_joint">
+        <command_interface name="velocity">
+            <param name="min">-1</param>
+            <param name="max">1</param>
+          </command_interface>
+          <state_interface name="position"/>
+          <state_interface name="velocity"/>
+      </joint>
+    </ros2_control>
+    <!-- Calling the pluging that will parse the ros2_control tags -->
+    <xacro:unless value="$(arg use_fake_components)">
+      <gazebo>
+        <plugin filename="libgazebo_ros2_control.so" name="gazebo_ros2_control">
+          <parameters>$(find zuuu_description)/config/zuuu_controllers.yaml</parameters>
+        </plugin>
+      </gazebo>
+    </xacro:unless>
+  </xacro:if>
   <link name="imu_link">
     <visual>
@@ -224,5 +227,5 @@
       <plugin filename="libgazebo_ros_imu_sensor.so" name="imu_plugin">
         <ros>
-          <namespace>/demo</namespace>
+          <namespace></namespace>
           <remapping>~/out:=imu</remapping>
         </ros>
