Commit message: fixing typos, works as it used to

File: urdf/zuuu.ros2_control.xacro (robot description, xacro)
@@ -2,41 +2,40 @@
 <robot xmlns:xacro="http://www.ros.org/wiki/xacro">
   <xacro:macro name="zuuu_ros2_control" params="model prefix">
-    <xacro:if value="$(arg use_ros_control)">
-        <ros2_control name="zuuu_ros2_control" type="system">
-        <hardware>
-            <xacro:if value="$(arg use_fake_components)">
-            <plugin>fake_components/GenericSystem</plugin>
-            </xacro:if>
-            <xacro:unless value="$(arg use_fake_components)">
-            <plugin>gazebo_ros2_control/GazeboSystem</plugin>
-            </xacro:unless>
-        </hardware>
-        <joint name="drivewhl1_joint">
-            <command_interface name="velocity">
-                <param name="min">-1</param>
-                <param name="max">1</param>
-            </command_interface>
-            <state_interface name="position"/>
-            <state_interface name="velocity"/>
-        </joint>
-        <joint name="drivewhl2_joint">
-            <command_interface name="velocity">
-                <param name="min">-1</param>
-                <param name="max">1</param>
-            </command_interface>
-            <state_interface name="position"/>
-            <state_interface name="velocity"/>
-        </joint>
-        <joint name="drivewhl3_joint">
-            <command_interface name="velocity">
-                <param name="min">-1</param>
-                <param name="max">1</param>
-            </command_interface>
-            <state_interface name="position"/>
-            <state_interface name="velocity"/>
-        </joint>
-        </ros2_control>
-        <!-- Calling the pluging that will parse the ros2_control tags -->
+    <ros2_control name="zuuu_ros2_control" type="system">
+    <hardware>
+        <xacro:if value="$(arg use_fake_components)">
+        <plugin>fake_components/GenericSystem</plugin>
+        </xacro:if>
         <xacro:unless value="$(arg use_fake_components)">
+        <plugin>gazebo_ros2_control/GazeboSystem</plugin>
+        </xacro:unless>
+    </hardware>
+    <joint name="drivewhl1_joint">
+        <command_interface name="velocity">
+            <param name="min">-1</param>
+            <param name="max">1</param>
+        </command_interface>
+        <state_interface name="position"/>
+        <state_interface name="velocity"/>
+    </joint>
+    <joint name="drivewhl2_joint">
+        <command_interface name="velocity">
+            <param name="min">-1</param>
+            <param name="max">1</param>
+        </command_interface>
+        <state_interface name="position"/>
+        <state_interface name="velocity"/>
+    </joint>
+    <joint name="drivewhl3_joint">
+        <command_interface name="velocity">
+            <param name="min">-1</param>
+            <param name="max">1</param>
+        </command_interface>
+        <state_interface name="position"/>
+        <state_interface name="velocity"/>
+    </joint>
+    </ros2_control>
+    <!-- Calling the pluging that will parse the ros2_control tags -->
+    <xacro:unless value="$(arg use_fake_components)">
         <gazebo>
             <plugin filename="libgazebo_ros2_control.so" name="gazebo_ros2_control">
@@ -44,6 +43,5 @@
             </plugin>
         </gazebo>
-        </xacro:unless>
-    </xacro:if>
+    </xacro:unless>
   </xacro:macro>
 </robot>

File: urdf/zuuu.urdf.xacro (robot description, xacro)
@@ -4,5 +4,5 @@
   <xacro:arg name="model" default="" />
   <xacro:arg name="use_gazebo" default="true"/>
-  <xacro:arg name="use_fake_components" default="false"/>
+  <xacro:arg name="use_fake_components" default="true"/>
   <xacro:arg name="use_fixed_wheels" default="true"/>
   <xacro:arg name="use_ros_control" default="true"/>
@@ -19,6 +19,6 @@
     <xacro:zuuu_gazebo model="$(arg model)" prefix="$(arg prefix)" />
   </xacro:if>
-  <xacro:zuuu_ros2_control
-    model="$(arg model)"
-    prefix="$(arg prefix)"/>
+  <xacro:if value="$(arg use_ros_control)">
+    <xacro:zuuu_ros2_control model="$(arg model)" prefix="$(arg prefix)"/>
+  </xacro:if>
 </robot>
