Commit message: Fragmenting files into urdf, gazebo and ros2_control

File: urdf/zuuu_description.urdf.xacro (robot description, xacro)
@@ -1,85 +1,103 @@
 <?xml version="1.0"?>
 <robot name="zuuu" xmlns:xacro="http://ros.org/wiki/xacro">
-  <xacro:arg name="use_fake_components" default="false"/>
-  <xacro:arg name="use_fixed_wheels" default="true"/>
-  <xacro:arg name="use_ros_control" default="true"/>
-  <!-- Define robot constants -->
-  <xacro:property name="base_radius" value="0.16"/>
-  <xacro:property name="base_top_height" value="0.1425"/>
-  <xacro:property name="base_depth" value="0.07"/>
-  <xacro:property name="wheel_radius" value="0.105"/>
-  <xacro:property name="wheel_width" value="0.035"/>
-  <xacro:property name="wheel_radial_dist" value="0.1805"/>
-  <xacro:property name="wheel_zoff" value="0.20"/>
-  <xacro:property name="global_damping" value="0.5"/>
-  <xacro:property name="global_friction" value="0.1"/>
-  <!-- Define some commonly used intertial properties  -->
-  <xacro:macro name="box_inertia" params="m w h d">
-    <inertial>
-      <origin xyz="0 0 0" rpy="${pi/2} 0 ${pi/2}"/>
-      <mass value="${m}"/>
-      <inertia ixx="${(m/12) * (h*h + d*d)}" ixy="0.0" ixz="0.0" iyy="${(m/12) * (w*w + d*d)}" iyz="0.0" izz="${(m/12) * (w*w + h*h)}"/>
-    </inertial>
-  </xacro:macro>
-  <xacro:macro name="cylinder_inertia" params="m r h">
-    <inertial>
-      <origin xyz="0 0 0" rpy="${pi/2} 0 0" />
-      <mass value="${m}"/>
-      <inertia ixx="${(m/12) * (3*r*r + h*h)}" ixy = "0" ixz = "0" iyy="${(m/12) * (3*r*r + h*h)}" iyz = "0" izz="${(m/2) * (r*r)}"/>
-    </inertial>
-  </xacro:macro>
-  <xacro:macro name="sphere_inertia" params="m r">
-    <inertial>
-      <mass value="${m}"/>
-      <inertia ixx="${(2/5) * m * (r*r)}" ixy="0.0" ixz="0.0" iyy="${(2/5) * m * (r*r)}" iyz="0.0" izz="${(2/5) * m * (r*r)}"/>
-    </inertial>
-  </xacro:macro>
-  <!-- Robot Footprint -->
-  <link name="base_footprint"/>
-  <joint name="base_footprint_joint" type="fixed">
-    <origin rpy="0 0 0" xyz="0 0 0"/>
-    <axis xyz="0 0 ${(base_top_height-base_depth/2)}"/>
-    <!-- <joint_properties damping="${global_damping}" friction="${global_friction}"/> -->
-    <parent link="base_footprint"/>
-    <child link="base_link"/>
-  </joint>
-  <!-- Robot Base -->
-  <link name="base_link">
-    <visual>
-      <geometry>
-        <cylinder radius="${base_radius}" length="${base_depth}"/>
-      </geometry>
-      <material name="Cyan">
-        <color rgba="0 1.0 1.0 1.0"/>
-      </material>
-    </visual>
-    <collision>
-      <geometry>
-        <cylinder radius="${base_radius}" length="${base_depth}"/>
-      </geometry>
-    </collision>
-    <xacro:cylinder_inertia m="20" r="${base_radius}" h="${base_depth}"/>
-  </link>
-  <!-- Wheels -->
-  <xacro:macro name="wheel" params="prefix yaw_angle">
-    <link name="${prefix}_link">
-      <visual>
-        <origin xyz="0 0 0" rpy="${pi/2} 0 0"/>
-        <geometry>
+  <xacro:macro name="zuuu" params="model prefix">
+    <!-- Define robot constants -->
+    <xacro:property name="base_radius" value="0.16"/>
+    <xacro:property name="base_top_height" value="0.1425"/>
+    <xacro:property name="base_depth" value="0.07"/>
+    <xacro:property name="wheel_radius" value="0.105"/>
+    <xacro:property name="wheel_width" value="0.035"/>
+    <xacro:property name="wheel_radial_dist" value="0.1805"/>
+    <xacro:property name="wheel_zoff" value="0.20"/>
+    <xacro:property name="global_damping" value="0.5"/>
+    <xacro:property name="global_friction" value="0.1"/>
+    <!-- Define some commonly used intertial properties  -->
+    <xacro:macro name="box_inertia" params="m w h d">
+      <inertial>
+        <origin xyz="0 0 0" rpy="${pi/2} 0 ${pi/2}"/>
+        <mass value="${m}"/>
+        <inertia ixx="${(m/12) * (h*h + d*d)}" ixy="0.0" ixz="0.0" iyy="${(m/12) * (w*w + d*d)}" iyz="0.0" izz="${(m/12) * (w*w + h*h)}"/>
+      </inertial>
+    </xacro:macro>
+    <xacro:macro name="cylinder_inertia" params="m r h">
+      <inertial>
+        <origin xyz="0 0 0" rpy="${pi/2} 0 0" />
+        <mass value="${m}"/>
+        <inertia ixx="${(m/12) * (3*r*r + h*h)}" ixy = "0" ixz = "0" iyy="${(m/12) * (3*r*r + h*h)}" iyz = "0" izz="${(m/2) * (r*r)}"/>
+      </inertial>
+    </xacro:macro>
+    <xacro:macro name="sphere_inertia" params="m r">
+      <inertial>
+        <mass value="${m}"/>
+        <inertia ixx="${(2/5) * m * (r*r)}" ixy="0.0" ixz="0.0" iyy="${(2/5) * m * (r*r)}" iyz="0.0" izz="${(2/5) * m * (r*r)}"/>
+      </inertial>
+    </xacro:macro>
+    <!-- Robot Footprint -->
+    <link name="base_footprint"/>
+    <joint name="base_footprint_joint" type="fixed">
+      <origin rpy="0 0 0" xyz="0 0 0"/>
+      <axis xyz="0 0 ${(base_top_height-base_depth/2)}"/>
+      <!-- <joint_properties damping="${global_damping}" friction="${global_friction}"/> -->
+      <parent link="base_footprint"/>
+      <child link="base_link"/>
+    </joint>
+    <!-- Robot Base -->
+    <link name="base_link">
+      <visual>
+        <geometry>
+          <cylinder radius="${base_radius}" length="${base_depth}"/>
+        </geometry>
+        <material name="Cyan">
+          <color rgba="0 1.0 1.0 1.0"/>
+        </material>
+      </visual>
+      <collision>
+        <geometry>
+          <cylinder radius="${base_radius}" length="${base_depth}"/>
+        </geometry>
+      </collision>
+      <xacro:cylinder_inertia m="20" r="${base_radius}" h="${base_depth}"/>
+    </link>
+    <!-- Wheels -->
+    <xacro:macro name="wheel" params="prefix yaw_angle">
+      <link name="${prefix}_link">
+        <visual>
+          <origin xyz="0 0 0" rpy="${pi/2} 0 0"/>
+          <geometry>
+              <cylinder radius="${wheel_radius}" length="${wheel_width}"/>
+              <box size="${wheel_radius} ${wheel_radius} ${wheel_width+0.02}"/>
+          </geometry>
+          <material name="Bricks"></material>
+        </visual>
+        <collision>
+          <origin xyz="0 0 0" rpy="${pi/2} 0 0"/>
+          <geometry>
             <cylinder radius="${wheel_radius}" length="${wheel_width}"/>
-            <box size="${wheel_radius} ${wheel_radius} ${wheel_width+0.02}"/>
-        </geometry>
-        <material name="Bricks"></material>
-      </visual>
-      <collision>
-        <origin xyz="0 0 0" rpy="${pi/2} 0 0"/>
-        <geometry>
-          <cylinder radius="${wheel_radius}" length="${wheel_width}"/>
-        </geometry>
-      </collision>
-      <xacro:cylinder_inertia m="0.5" r="${wheel_radius}" h="${wheel_width}"/>
-    </link>
-    <xacro:if value="$(arg use_fixed_wheels)">
-        <joint name="${prefix}_joint" type="fixed">
+          </geometry>
+        </collision>
+        <xacro:cylinder_inertia m="0.5" r="${wheel_radius}" h="${wheel_width}"/>
+      </link>
+      <xacro:if value="$(arg use_fixed_wheels)">
+          <joint name="${prefix}_joint" type="fixed">
+            <parent link="base_link"/>
+            <child link="${prefix}_link"/>
+            <origin xyz="${wheel_radial_dist*cos(yaw_angle)} ${-wheel_radial_dist*sin(yaw_angle)} ${-((base_top_height-base_depth/2)- wheel_radius)}" rpy="0 0 ${pi/2-yaw_angle}"/>
+            <axis xyz="0 1 0"/>
+            <joint_properties damping="${global_damping}" friction="${global_friction}"/>
+          </joint>
+          <!-- No friction because we suck and everything is lame -->
+          <gazebo reference="${prefix}_link">
+            <mu1 value="0.0"/>
+            <mu2 value="0.0"/>
+            <kp value="10000000.0" />
+            <kd value="1.0" />
+            <fdir1 value="1 0 0"/>
+            <maxVel>1.0</maxVel>
+            <minDepth>0.0</minDepth>
+            <turnGravityOff>false</turnGravityOff>
+          </gazebo>
+      </xacro:if>
+      <xacro:unless value="$(arg use_fixed_wheels)">
+        <joint name="${prefix}_joint" type="continuous">
           <parent link="base_link"/>
           <child link="${prefix}_link"/>
@@ -88,331 +106,109 @@
           <joint_properties damping="${global_damping}" friction="${global_friction}"/>
         </joint>
-        <!-- No friction because we suck and everything is lame -->
+        <!-- Physics because we're smart and handsome -->
         <gazebo reference="${prefix}_link">
-          <mu1 value="0.0"/>
+          <mu1 value="1.0"/>
           <mu2 value="0.0"/>
           <kp value="10000000.0" />
           <kd value="1.0" />
           <fdir1 value="1 0 0"/>
-          <maxVel>1.0</maxVel>
-          <minDepth>0.0</minDepth>
+          <maxVel>5.0</maxVel>
+          <minDepth>0.002</minDepth>
           <turnGravityOff>false</turnGravityOff>
         </gazebo>
-    </xacro:if>
-    <xacro:unless value="$(arg use_fixed_wheels)">
-      <joint name="${prefix}_joint" type="continuous">
-        <parent link="base_link"/>
-        <child link="${prefix}_link"/>
-        <origin xyz="${wheel_radial_dist*cos(yaw_angle)} ${-wheel_radial_dist*sin(yaw_angle)} ${-((base_top_height-base_depth/2)- wheel_radius)}" rpy="0 0 ${pi/2-yaw_angle}"/>
-        <axis xyz="0 1 0"/>
-        <joint_properties damping="${global_damping}" friction="${global_friction}"/>
+      </xacro:unless>
+      <!-- Just so that we can see the wheels turn when they turn -->
+      <link name="${prefix}_extra_link">
+        <visual>
+          <origin xyz="0 0 0" rpy="${pi/2} 0 0"/>
+          <geometry>
+              <box size="${wheel_radius} ${wheel_radius} ${wheel_width+0.02}"/>
+          </geometry>
+        </visual>
+      </link>
+      <joint name="${prefix}_extra_joint" type="fixed">
+        <origin rpy="0 0 0" xyz="0 0 0"/>
+        <axis xyz="0 0 0"/>
+        <parent link="${prefix}_link"/>
+        <child link="${prefix}_extra_link"/>
       </joint>
-      <!-- Physics because we're smart and handsome -->
-      <gazebo reference="${prefix}_link">
-        <mu1 value="1.0"/>
-        <mu2 value="0.0"/>
-        <kp value="10000000.0" />
-        <kd value="1.0" />
-        <fdir1 value="1 0 0"/>
-        <maxVel>5.0</maxVel>
-        <minDepth>0.002</minDepth>
-        <turnGravityOff>false</turnGravityOff>
-      </gazebo>
-    </xacro:unless>
-    <!-- Just so that we can see the wheels turn when they turn -->
-    <link name="${prefix}_extra_link">
-      <visual>
-        <origin xyz="0 0 0" rpy="${pi/2} 0 0"/>
-        <geometry>
-            <box size="${wheel_radius} ${wheel_radius} ${wheel_width+0.02}"/>
-        </geometry>
-      </visual>
-    </link>
-    <joint name="${prefix}_extra_joint" type="fixed">
-      <origin rpy="0 0 0" xyz="0 0 0"/>
-      <axis xyz="0 0 0"/>
-      <parent link="${prefix}_link"/>
-      <child link="${prefix}_extra_link"/>
+    </xacro:macro>
+    <!-- Wheel 1 at the back, 2 on the right, 3 on the left -->
+    <xacro:wheel prefix="drivewhl1" yaw_angle="${pi/3}" />
+    <xacro:wheel prefix="drivewhl2" yaw_angle="${5*pi/3}" />
+    <xacro:wheel prefix="drivewhl3" yaw_angle="${pi}" />
+    <link name="imu_link">
+      <visual>
+        <geometry>
+          <box size="0.1 0.1 0.02"/>
+        </geometry>
+      </visual>
+      <collision>
+        <geometry>
+          <box size="0.1 0.1 0.1"/>
+        </geometry>
+      </collision>
+      <xacro:box_inertia m="0.1" w="0.1" d="0.1" h="0.1"/>
+    </link>
+    <joint name="imu_joint" type="fixed">
+      <parent link="base_link"/>
+      <child link="imu_link"/>
+      <origin xyz="0 0 0.01"/>
+    </joint>
+  <link name="lidar_link">
+      <inertial>
+        <origin xyz="0 0 0" rpy="0 0 0"/>
+        <mass value="0.125"/>
+        <inertia ixx="0.001"  ixy="0"  ixz="0" iyy="0.001" iyz="0" izz="0.001" />
+      </inertial>
+      <collision>
+        <origin xyz="0 0 0" rpy="0 0 0"/>
+        <geometry>
+          <cylinder radius="0.0508" length="0.055"/>
+        </geometry>
+      </collision>
+      <visual>
+        <origin xyz="0 0 0" rpy="0 0 0"/>
+        <geometry>
+          <cylinder radius="0.0508" length="0.055"/>
+        </geometry>
+      </visual>
+    </link>
+    <joint name="lidar_joint" type="fixed">
+      <parent link="base_link"/>
+      <child link="lidar_link"/>
+      <!-- <origin xyz="0.155 0 0.2" rpy="0 0 0"/> -->
+      <origin xyz="0.155 0 ${-(base_top_height-base_depth/2)+base_top_height+0.105}" rpy="0 0 0"/>
+    </joint>
+    <link name="camera_link">
+      <visual>
+        <origin xyz="0 0 0" rpy="0 0 0"/>
+        <geometry>
+          <box size="0.015 0.130 0.022"/>
+        </geometry>
+      </visual>
+      <collision>
+        <origin xyz="0 0 0" rpy="0 0 0"/>
+        <geometry>
+          <box size="0.015 0.130 0.022"/>
+        </geometry>
+      </collision>
+      <inertial>
+        <origin xyz="0 0 0" rpy="0 0 0"/>
+        <mass value="0.035"/>
+        <inertia ixx="0.001"  ixy="0"  ixz="0" iyy="0.001" iyz="0" izz="0.001" />
+      </inertial>
+    </link>
+    <joint name="camera_joint" type="fixed">
+      <parent link="base_link"/>
+      <child link="camera_link"/>
+      <origin xyz="0.155 0 0.5" rpy="0 0 0"/>
+    </joint>
+    <link name="camera_depth_frame"/>
+    <joint name="camera_depth_joint" type="fixed">
+      <origin xyz="0 0 0" rpy="${-pi/2} 0 ${-pi/2}"/>
+      <parent link="camera_link"/>
+      <child link="camera_depth_frame"/>
     </joint>
   </xacro:macro>
-  <!-- Wheel 1 at the back, 2 on the right, 3 on the left -->
-  <xacro:wheel prefix="drivewhl1" yaw_angle="${pi/3}" />
-  <xacro:wheel prefix="drivewhl2" yaw_angle="${5*pi/3}" />
-  <xacro:wheel prefix="drivewhl3" yaw_angle="${pi}" />
-  <gazebo>
-    <plugin name="object_controller" filename="libgazebo_ros_planar_move.so">
-      <commandTopic>cmd_vel</commandTopic>
-      <odometryTopic>odom</odometryTopic>
-      <robotNamespace> </robotNamespace>
-      <!-- Set control loop update rate -->
-      <odometryRate>100</odometryRate>
-      <!-- Set odom publish rate -->
-      <publish_rate>100</publish_rate>
-      <!-- Set if odom required -->
-      <publish_odom>true</publish_odom>
-      <publish_odom_tf>true</publish_odom_tf>
-      <!-- Frame IDs -->
-      <odometryFrame>odom</odometryFrame>
-      <robotBaseFrame>base_link</robotBaseFrame>
-      <!-- Set odom covariance -->
-      <covariance_x>0.0001</covariance_x>
-      <covariance_y>0.0001</covariance_y>
-      <covariance_yaw>0.01</covariance_yaw>
-    </plugin>
-  </gazebo>
-  <xacro:if value="$(arg use_ros_control)">
-    <ros2_control name="zuuu_ros2_control" type="system">
-      <hardware>
-        <xacro:if value="$(arg use_fake_components)">
-          <plugin>fake_components/GenericSystem</plugin>
-        </xacro:if>
-        <xacro:unless value="$(arg use_fake_components)">
-          <plugin>gazebo_ros2_control/GazeboSystem</plugin>
-        </xacro:unless>
-      </hardware>
-      <joint name="drivewhl1_joint">
-        <command_interface name="velocity">
-            <param name="min">-1</param>
-            <param name="max">1</param>
-          </command_interface>
-          <state_interface name="position"/>
-          <state_interface name="velocity"/>
-      </joint>
-      <joint name="drivewhl2_joint">
-        <command_interface name="velocity">
-            <param name="min">-1</param>
-            <param name="max">1</param>
-          </command_interface>
-          <state_interface name="position"/>
-          <state_interface name="velocity"/>
-      </joint>
-      <joint name="drivewhl3_joint">
-        <command_interface name="velocity">
-            <param name="min">-1</param>
-            <param name="max">1</param>
-          </command_interface>
-          <state_interface name="position"/>
-          <state_interface name="velocity"/>
-      </joint>
-    </ros2_control>
-    <!-- Calling the pluging that will parse the ros2_control tags -->
-    <xacro:unless value="$(arg use_fake_components)">
-      <gazebo>
-        <plugin filename="libgazebo_ros2_control.so" name="gazebo_ros2_control">
-          <parameters>$(find zuuu_description)/config/zuuu_controllers.yaml</parameters>
-        </plugin>
-      </gazebo>
-    </xacro:unless>
-  </xacro:if>
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
Commit message: Applying Z-delta on LIDAR based on the new hardware change

File: urdf/zuuu_description.urdf.xacro (robot description, xacro)
@@ -156,5 +156,5 @@
       <origin xyz="0 0 0.01"/>
     </joint>
-  <link name="lidar_link">
+    <link name="lidar_link">
       <inertial>
         <origin xyz="0 0 0" rpy="0 0 0"/>
@@ -179,5 +179,6 @@
       <child link="lidar_link"/>
       <!-- <origin xyz="0.155 0 0.2" rpy="0 0 0"/> -->
-      <origin xyz="0.155 0 ${-(base_top_height-base_depth/2)+base_top_height+0.105}" rpy="0 0 0"/>
+      <!-- The -0.0129 were added on 22 pril 2022 for the second version of Zuuu. The 2mm pads are not taken into account -->
+      <origin xyz="0.155 0 ${-(base_top_height-base_depth/2)+base_top_height+0.105 -0.0129}" rpy="0 0 0"/>
     </joint>
     <link name="camera_link">

Commit message: adding a monolithic 3D reachy mobil daee

File: urdf/zuuu_description.urdf.xacro (robot description, xacro)
@@ -52,4 +52,10 @@
         </material>
       </visual>
+      <visual>
+        <origin xyz="0 0 ${(-base_top_height+base_depth/2)}" rpy="0 0 0"/>
+        <geometry>
+          <mesh filename="file://$(find zuuu_description)/meshes/reachy_mobile_pauvre.dae"/>
+        </geometry>
+      </visual>
       <collision>
         <geometry>
@@ -62,5 +68,5 @@
     <xacro:macro name="wheel" params="prefix yaw_angle">
       <link name="${prefix}_link">
-        <visual>
+        <!-- <visual>
           <origin xyz="0 0 0" rpy="${pi/2} 0 0"/>
           <geometry>
@@ -69,5 +75,5 @@
           </geometry>
           <material name="Bricks"></material>
-        </visual>
+        </visual> -->
         <collision>
           <origin xyz="0 0 0" rpy="${pi/2} 0 0"/>
@@ -120,10 +126,10 @@
       <!-- Just so that we can see the wheels turn when they turn -->
       <link name="${prefix}_extra_link">
-        <visual>
+        <!-- <visual>
           <origin xyz="0 0 0" rpy="${pi/2} 0 0"/>
           <geometry>
               <box size="${wheel_radius} ${wheel_radius} ${wheel_width+0.02}"/>
           </geometry>
-        </visual>
+        </visual> -->
       </link>
       <joint name="${prefix}_extra_joint" type="fixed">

Commit message: minor description update

File: urdf/zuuu_description.urdf.xacro (robot description, xacro)
@@ -44,5 +44,5 @@
     <!-- Robot Base -->
     <link name="base_link">
-      <visual>
+      <!-- <visual>
         <geometry>
           <cylinder radius="${base_radius}" length="${base_depth}"/>
@@ -51,5 +51,5 @@
           <color rgba="0 1.0 1.0 1.0"/>
         </material>
-      </visual>
+      </visual> -->
       <visual>
         <origin xyz="0 0 ${(-base_top_height+base_depth/2)}" rpy="0 0 0"/>
@@ -145,9 +145,9 @@
     <xacro:wheel prefix="drivewhl3" yaw_angle="${pi}" />
     <link name="imu_link">
-      <visual>
+      <!-- <visual>
         <geometry>
           <box size="0.1 0.1 0.02"/>
         </geometry>
-      </visual>
+      </visual> -->
       <collision>
         <geometry>
@@ -174,10 +174,10 @@
         </geometry>
       </collision>
-      <visual>
+      <!-- <visual>
         <origin xyz="0 0 0" rpy="0 0 0"/>
         <geometry>
           <cylinder radius="0.0508" length="0.055"/>
         </geometry>
-      </visual>
+      </visual> -->
     </link>
     <joint name="lidar_joint" type="fixed">
@@ -189,10 +189,10 @@
     </joint>
     <link name="camera_link">
-      <visual>
+      <!-- <visual>
         <origin xyz="0 0 0" rpy="0 0 0"/>
         <geometry>
           <box size="0.015 0.130 0.022"/>
         </geometry>
-      </visual>
+      </visual> -->
       <collision>
         <origin xyz="0 0 0" rpy="0 0 0"/>
